Commit message: nova versão do rosbot3_description

File: urdf/rosbot3.xacro (robot description, xacro)
@@ -7,10 +7,11 @@
 <robot name="rosbot3" xmlns:xacro="http://www.ros.org/wiki/xacro">
   <xacro:include filename="$(find rosbot3_description)/urdf/ugv02.xacro"/>
-  <xacro:property name="payload_base_length" value="${156.22 * M}"/>
-  <xacro:property name="payload_base_width" value="${159.96 * M}"/>
-  <xacro:property name="payload_base_height" value="${42.7 * M}"/>
-  <xacro:property name="lidar_side" value="${45.61 * M}"/>
-  <xacro:property name="lidar_height" value="${37.6 * M}"/>
-  <xacro:solid_block
+  <xacro:property name="payload_base_length" value="${200.0 * M}"/> <!-- comprimento da base para sensores -->
+  <xacro:property name="payload_base_width" value="${223.0 * M}"/> <!-- largura da base para sensores -->
+  <xacro:property name="payload_base_height" value="${1.0 * M}"/> <!-- altura da base para sensores -->
+  <xacro:property name="lidar_radius" value="${10.0 * M}"/> <!-- raio do cilindro do LiDAR -->
+  <xacro:property name="lidar_height" value="${38.0 * M}"/> <!-- altura do LiDAR -->
+  <!-- Corpo principal do robô -->
+  <xacro:solid_block_red
     name="payload_base"
     size_x="${payload_base_length}"
@@ -18,4 +19,5 @@
     size_z="${payload_base_height}"
   />
+<!-- Junta fixa conectando a base de carga ao corpo principal -->
   <xacro:joint_fixed
     parent="body"
@@ -29,8 +31,8 @@
     x="${0.5 * payload_base_length}"
   />
-  <xacro:solid_block
+  <xacro:solid_block_black
     name="lidar"
-    size_x="${lidar_side}"
-    size_y="${lidar_side}"
+    size_x="${lidar_radius}"
+    size_y="${lidar_radius}"
     size_z="${lidar_height}"
   />

File: urdf/ugv02.xacro (robot description, xacro)
@@ -1,52 +1,69 @@
 <?xml version="1.0" encoding="utf-8"?>
 <!--
-  Description of the Waveshare UGV02 mobile base upon which ROSBOT3 is built.
-  Author: Helio Perroni Filho
+  Modelo simplificado do Waveshare UGV02 (ROSelito) com 4 rodas
+  - Duas dianteiras e duas traseiras
+  - base_link é o link raiz físico (com massa/inércia)
+  Autor original: Helio Perroni Filho
+  Adaptado por: Vito Rodrigues Franzosi
 -->
 <robot xmlns:xacro="http://www.ros.org/wiki/xacro">
+  <!-- Inclui primitivas e macros comuns -->
   <xacro:include filename="$(find ros_commons)/urdf/domain.xacro"/>
+  <!-- Escala (mm -> m) -->
   <xacro:property name="M" value="0.001"/>
-  <xacro:property name="ground_clearance" value="${25.13 * M}"/>
-  <xacro:property name="overall_height" value="${93.88 * M}"/>
-  <xacro:property name="fender_height" value="${10.0 * M}"/>
-  <xacro:property name="wheel_separation" value="${126.0 * M}"/>
-  <xacro:property name="wheel_diameter" value="${overall_height - fender_height}"/>
-  <xacro:property name="wheelbase" value="${252.45 * M - wheel_diameter}"/>
-  <xacro:property name="wheel_radius" value="${0.5 * wheel_diameter}"/>
-  <xacro:property name="wheel_thickness" value="${50.21 * M}"/>
-  <xacro:property name="fender_length" value="${214.04 * M}"/>
-  <xacro:property name="fender_thickness" value="${3.0 * M}"/>
-  <xacro:property name="fender_top_gap" value="${1.0 * M}"/>
-  <xacro:property name="fender_side_gap" value="${5.0 * M}"/>
-  <xacro:property name="body_length" value="${243.18 * M}"/>
-  <xacro:property name="body_width" value="${126.0 * M}"/>
-  <xacro:property name="body_height" value="${wheel_diameter - ground_clearance + fender_top_gap + fender_thickness}"/>
-  <xacro:property name="fender_top_width" value="${body_width + 2.0 * (wheel_thickness + fender_side_gap)}"/>
-  <xacro:property name="fender_side_width" value="${wheel_radius + fender_thickness + fender_top_gap}"/>
-  <xacro:property name="fender_side_y_offset" value="${0.5 * (fender_top_width + fender_thickness)}"/>
-  <xacro:property name="fender_side_z_offset" value="${0.5 * (fender_thickness - fender_side_width)}"/>
-  <xacro:property name="wheel_axle_z_offset" value="${wheel_radius - 0.5 * body_height - ground_clearance}"/>
-  <xacro:macro
-    name="wheels"
-    params="position"
-  >
+  <!-- Dimensões principais -->
+  <xacro:property name="ground_clearance" value="${23.0 * M}"/> <!-- distância do chão até a parte mais baixa do corpo -->
+  <xacro:property name="overall_height" value="${103.0 * M}"/>  <!-- altura total do robô -->
+  <xacro:property name="fender_height" value="${10.0 * M}"/>  <!-- altura dos para-lamas acima do corpo -->
+  <xacro:property name="wheel_separation" value="${126.0 * M}"/> <!-- distância entre rodas esquerda e direita -->
+  <xacro:property name="wheel_diameter" value="${84.0 * M}"/> <!-- diâmetro das rodas -->
+  <xacro:property name="wheel_radius" value="${0.5 * wheel_diameter}"/> <!-- raio das rodas -->
+  <xacro:property name="wheel_thickness" value="${50.21 * M}"/> <!-- espessura das rodas -->
+  <xacro:property name="wheelbase" value="${104.0 * M}"/> <!-- distância entre eixos dianteiro e traseiro -->
+  <xacro:property name="body_length" value="${200.0 * M}"/> <!-- comprimento total do corpo -->
+  <xacro:property name="body_width" value="${126.0 * M + wheel_thickness - 10.0 * M}"/> <!-- largura total do corpo -->
+  <xacro:property name="body_height" value="${103.0 * M - ground_clearance + 0.004}"/> <!-- altura do corpo (ajuste de 4mm para evitar colisão com o chão) -->
+  <xacro:property name="wheel_axle_z_offset" value="${wheel_radius - 0.5 * body_height - ground_clearance}"/> <!-- altura do eixo das rodas em relação à base do corpo -->
+  <!-- === Definir base_link (link raiz físico) === -->
+  <link name="base_link">
+    <inertial>
+      <!-- massa total aproximada do robô (ajuste se quiser) -->
+      <mass value="8.0"/>
+      <origin xyz="0 0 0" rpy="0 0 0"/>
+      <!-- tensores de inércia simplificados (aprox.) -->
+      <inertia ixx="0.12" iyy="0.18" izz="0.10" ixy="0.0" ixz="0.0" iyz="0.0"/>
+    </inertial>
+    <visual>
+      <origin xyz="0 0 0" rpy="0 0 0"/>
+      <geometry>
+        <!-- pequena caixa representando a base (opcional, apenas para colisão/visual) -->
+        <box size="${0.01} ${0.01} ${0.01}"/>
+      </geometry>
+    </visual>
+    <collision>
+      <origin xyz="0 0 0" rpy="0 0 0"/>
+      <geometry>
+        <box size="${0.01} ${0.01} ${0.01}"/>
+      </geometry>
+    </collision>
+  </link>
+  <!-- === Macro para rodas === -->
+  <xacro:macro name="wheels" params="position x_offset">
+    <xacro:solid_cylinder
+      name="wheel_${position}_axle"
+      length="${wheel_separation}"
+      radius="0.005"
+      roll="${90.0 * DEG}"/>
+    <!-- rodas esquerda/direita como cilindros visuais e com joints contínuos -->
     <xacro:solid_cylinder
       name="wheel_${position}_left"
       length="${wheel_thickness}"
       radius="${wheel_radius}"
-      roll="${90.0 * DEG}"
-    />
+      roll="${90.0 * DEG}"/>
     <xacro:solid_cylinder
       name="wheel_${position}_right"
       length="${wheel_thickness}"
       radius="${wheel_radius}"
-      roll="${90.0 * DEG}"
-    />
-    <xacro:solid_cylinder
-      name="wheel_${position}_axle"
-      length="${wheel_separation}"
-      radius="0.005"
-      roll="${90.0 * DEG}"
-    />
+      roll="${90.0 * DEG}"/>
     <xacro:joint_continuous
       name="joint_wheel_${position}_left"
@@ -54,6 +71,5 @@
       child="wheel_${position}_left"
       y="${(wheel_separation + wheel_thickness) * 0.5}"
-      axis="0 1 0"
-    />
+      axis="0 1 0"/>
     <xacro:joint_continuous
       name="joint_wheel_${position}_right"
@@ -61,73 +77,42 @@
       child="wheel_${position}_right"
       y="${(wheel_separation + wheel_thickness) * -0.5}"
-      axis="0 1 0"
-    />
+      axis="0 1 0"/>
+    <!-- junta fixa para posicionar o axle relativo ao pai (sera usada abaixo) -->
+    <!-- (não cria link adicional aqui — a junta será criada externamente quando necessário) -->
   </xacro:macro>
-  <xacro:wheels position="front"/>
-  <xacro:wheels position="center"/>
-  <xacro:wheels position="rear"/>
+  <!-- Instancia rodas (front e rear). Fornecemos x_offset apenas para documentação; posicionamento feito por joints -->
+  <xacro:wheels position="front" x_offset="${0.5 * wheelbase}"/>
+  <xacro:wheels position="rear"  x_offset="${-0.5 * wheelbase}"/>
+  <!-- Corpo do robô (visual) -->
   <xacro:solid_block
     name="body"
     size_x="${body_length}"
     size_y="${body_width}"
-    size_z="${body_height}"
-  />
-  <xacro:solid_block
-    name="fenders_top"
-    size_x="${fender_length}"
-    size_y="${fender_top_width}"
-    size_z="${fender_thickness}"
-  />
-  <xacro:solid_block
-    name="fender_left"
-    size_x="${fender_length}"
-    size_y="${fender_thickness}"
-    size_z="${fender_side_width}"
-  />
-  <xacro:solid_block
-    name="fender_right"
-    size_x="${fender_length}"
-    size_y="${fender_thickness}"
-    size_z="${fender_side_width}"
-  />
+    size_z="${body_height}"/>
+  <!-- === Juntas e posicionamento === -->
+  <!-- Posiciona o body em relação ao base_link.
+       Queremos que a origem (0,0,0) do base_link coincida com o eixo traseiro.
+       Então deslocamos o body para frente em +0.5*wheelbase (corpo fica à frente da roda traseira).
+  -->
   <xacro:joint_fixed
+    name="joint_base_body"
+    parent="base_link"
+    child="body"
+    x="${0.5 * wheelbase}"
+    z="${ground_clearance + 0.5 * body_height}"/>
+  <!-- Posiciona o eixo traseiro relativo ao body (visto a partir do body) -->
+  <xacro:joint_fixed
+    name="joint_body_wheel_rear_axle"
     parent="body"
-    child="fenders_top"
-    z="${0.5 * (body_height - fender_thickness)}"
-  />
+    child="wheel_rear_axle"
+    x="${-0.5 * wheelbase}"
+    z="${wheel_axle_z_offset}"/>
+  <!-- Posiciona o eixo dianteiro relativo ao body -->
   <xacro:joint_fixed
-    parent="fenders_top"
-    child="fender_left"
-    y="${fender_side_y_offset}"
-    z="${fender_side_z_offset}"
-  />
-  <xacro:joint_fixed
-    parent="fenders_top"
-    child="fender_right"
-    y="${-fender_side_y_offset}"
-    z="${fender_side_z_offset}"
-  />
-  <xacro:joint_fixed
+    name="joint_body_wheel_front_axle"
     parent="body"
     child="wheel_front_axle"
     x="${0.5 * wheelbase}"
-    z="${wheel_axle_z_offset}"
-  />
-  <xacro:joint_fixed
-    parent="body"
-    child="wheel_center_axle"
-    z="${wheel_axle_z_offset}"
-  />
-  <xacro:joint_fixed
-    parent="body"
-    child="wheel_rear_axle"
-    x="${-0.5 * wheelbase}"
-    z="${wheel_axle_z_offset}"
-  />
-  <link name="base_link"/>
-  <xacro:joint_fixed
-    parent="base_link"
-    child="body"
-    z="${ground_clearance + 0.5 * body_height}"
-  />
+    z="${wheel_axle_z_offset}"/>
+  <!-- OBS: wheel_*_left/right já estão ligados aos respectivos axle via joint_continuous dentro da macro -->
 </robot>

Commit message: correções para atender as características do robot3

File: urdf/rosbot3.xacro (robot description, xacro)
@@ -2,16 +2,16 @@
 <!--
   Description of the ROSBOT3 robot.
-  Author: Vito Rodrigues Franzosi
+  Autor original: Helio Perroni Filho
+  Adaptado por: Vito Rodrigues Franzosi
   Date: 06.11.2025
 -->
 <robot name="rosbot3" xmlns:xacro="http://www.ros.org/wiki/xacro">
   <xacro:include filename="$(find rosbot3_description)/urdf/ugv02.xacro"/>
-  <xacro:property name="payload_base_length" value="${200.0 * M}"/> <!-- comprimento da base para sensores -->
-  <xacro:property name="payload_base_width" value="${223.0 * M}"/> <!-- largura da base para sensores -->
-  <xacro:property name="payload_base_height" value="${1.0 * M}"/> <!-- altura da base para sensores -->
-  <xacro:property name="lidar_radius" value="${10.0 * M}"/> <!-- raio do cilindro do LiDAR -->
-  <xacro:property name="lidar_height" value="${38.0 * M}"/> <!-- altura do LiDAR -->
-  <!-- Corpo principal do robô -->
-  <xacro:solid_block_red
+  <xacro:property name="payload_base_length" value="${156.22 * M}"/>
+  <xacro:property name="payload_base_width" value="${159.96 * M}"/>
+  <xacro:property name="payload_base_height" value="${42.7 * M}"/>
+  <xacro:property name="lidar_side" value="${45.61 * M}"/>
+  <xacro:property name="lidar_height" value="${37.6 * M}"/>
+  <xacro:solid_block
     name="payload_base"
     size_x="${payload_base_length}"
@@ -19,5 +19,4 @@
     size_z="${payload_base_height}"
   />
-<!-- Junta fixa conectando a base de carga ao corpo principal -->
   <xacro:joint_fixed
     parent="body"
@@ -31,8 +30,8 @@
     x="${0.5 * payload_base_length}"
   />
-  <xacro:solid_block_black
+  <xacro:solid_block
     name="lidar"
-    size_x="${lidar_radius}"
-    size_y="${lidar_radius}"
+    size_x="${lidar_side}"
+    size_y="${lidar_side}"
     size_z="${lidar_height}"
   />

File: urdf/ugv02.xacro (robot description, xacro)
@@ -6,64 +6,51 @@
   Autor original: Helio Perroni Filho
   Adaptado por: Vito Rodrigues Franzosi
+  Date: 06.11.2025
 -->
-<robot xmlns:xacro="http://www.ros.org/wiki/xacro">
-  <!-- Inclui primitivas e macros comuns -->
-  <xacro:include filename="$(find ros_commons)/urdf/domain.xacro"/>
-  <!-- Escala (mm -> m) -->
+<robot xmlns:xacro="http://www.ros.org/wiki/xacro"> <!-- Definição do namespace xacro -->
+  <xacro:include filename="$(find ros_commons)/urdf/domain.xacro"/> <!-- Inclui definições de primitivas geométricas -->
   <xacro:property name="M" value="0.001"/>
-  <!-- Dimensões principais -->
-  <xacro:property name="ground_clearance" value="${23.0 * M}"/> <!-- distância do chão até a parte mais baixa do corpo -->
-  <xacro:property name="overall_height" value="${103.0 * M}"/>  <!-- altura total do robô -->
-  <xacro:property name="fender_height" value="${10.0 * M}"/>  <!-- altura dos para-lamas acima do corpo -->
-  <xacro:property name="wheel_separation" value="${126.0 * M}"/> <!-- distância entre rodas esquerda e direita -->
-  <xacro:property name="wheel_diameter" value="${84.0 * M}"/> <!-- diâmetro das rodas -->
-  <xacro:property name="wheel_radius" value="${0.5 * wheel_diameter}"/> <!-- raio das rodas -->
-  <xacro:property name="wheel_thickness" value="${50.21 * M}"/> <!-- espessura das rodas -->
-  <xacro:property name="wheelbase" value="${104.0 * M}"/> <!-- distância entre eixos dianteiro e traseiro -->
-  <xacro:property name="body_length" value="${200.0 * M}"/> <!-- comprimento total do corpo -->
-  <xacro:property name="body_width" value="${126.0 * M + wheel_thickness - 10.0 * M}"/> <!-- largura total do corpo -->
-  <xacro:property name="body_height" value="${103.0 * M - ground_clearance + 0.004}"/> <!-- altura do corpo (ajuste de 4mm para evitar colisão com o chão) -->
-  <xacro:property name="wheel_axle_z_offset" value="${wheel_radius - 0.5 * body_height - ground_clearance}"/> <!-- altura do eixo das rodas em relação à base do corpo -->
-  <!-- === Definir base_link (link raiz físico) === -->
-  <link name="base_link">
-    <inertial>
-      <!-- massa total aproximada do robô (ajuste se quiser) -->
-      <mass value="8.0"/>
-      <origin xyz="0 0 0" rpy="0 0 0"/>
-      <!-- tensores de inércia simplificados (aprox.) -->
-      <inertia ixx="0.12" iyy="0.18" izz="0.10" ixy="0.0" ixz="0.0" iyz="0.0"/>
-    </inertial>
-    <visual>
-      <origin xyz="0 0 0" rpy="0 0 0"/>
-      <geometry>
-        <!-- pequena caixa representando a base (opcional, apenas para colisão/visual) -->
-        <box size="${0.01} ${0.01} ${0.01}"/>
-      </geometry>
-    </visual>
-    <collision>
-      <origin xyz="0 0 0" rpy="0 0 0"/>
-      <geometry>
-        <box size="${0.01} ${0.01} ${0.01}"/>
-      </geometry>
-    </collision>
-  </link>
-  <!-- === Macro para rodas === -->
-  <xacro:macro name="wheels" params="position x_offset">
+  <xacro:property name="ground_clearance" value="${23.0 * M}"/> <!-- Distância do solo até a parte mais baixa do corpo -->
+  <xacro:property name="overall_height" value="${103 * M}"/> <!-- Altura total do robô -->
+  <xacro:property name="fender_height" value="${10.0 * M}"/> <!-- Altura dos para-lamas -->
+  <xacro:property name="wheel_separation" value="${126.0 * M}"/> <!-- Distância entre as rodas esquerda e direita -->
+  <xacro:property name="wheel_diameter" value="${84.0 * M}"/> <!-- Diâmetro das rodas -->
+  <xacro:property name="wheelbase" value="${104.0 * M}"/> <!-- Distância entre os eixos dianteiro e traseiro -->
+  <xacro:property name="wheel_radius" value="${0.5 * wheel_diameter}"/> <!-- Raio das rodas -->
+  <xacro:property name="wheel_thickness" value="${50.21 * M}"/>  <!-- Espessura das rodas -->
+  <xacro:property name="fender_length" value="${200.0 * M}"/> <!-- Comprimento dos para-lamas -->
+  <xacro:property name="fender_thickness" value="${3.0 * M}"/> <!-- Espessura dos para-lamas -->
+  <xacro:property name="fender_top_width" value="${126.0 * M + wheel_thickness}"/> <!-- Largura do para-lama superior -->
+  <xacro:property name="body_length" value="${200.0 * M}"/> <!-- Comprimento do corpo do robô -->
+  <xacro:property name="body_width" value="${126.0 * M}"/>
+  <xacro:property name="body_height" value="${103.0 * M - ground_clearance + 0.004}"/> <!-- Altura do corpo do robô -->
+  <xacro:property name="wheel_axle_z_offset" value="${wheel_radius - 0.5 * body_height - ground_clearance}"/>  <!-- Deslocamento Z dos eixos das rodas -->
+  <!-- Definição das rodas -->
+  <xacro:macro
+    name="wheels"
+    params="position"
+  >
+    <!-- Definição das rodas esquerda, direita e do eixo -->
+    <xacro:solid_cylinder
+      name="wheel_${position}_left"
+      length="${wheel_thickness}"
+      radius="${wheel_radius}"
+      roll="${90.0 * DEG}"
+    />
+    <!-- Definição das rodas direita e do eixo -->
+    <xacro:solid_cylinder
+      name="wheel_${position}_right"
+      length="${wheel_thickness}"
+      radius="${wheel_radius}"
+      roll="${90.0 * DEG}"
+    />
+    <!-- Definição do eixo das rodas -->
     <xacro:solid_cylinder
       name="wheel_${position}_axle"
       length="${wheel_separation}"
       radius="0.005"
-      roll="${90.0 * DEG}"/>
-    <!-- rodas esquerda/direita como cilindros visuais e com joints contínuos -->
-    <xacro:solid_cylinder
-      name="wheel_${position}_left"
-      length="${wheel_thickness}"
-      radius="${wheel_radius}"
-      roll="${90.0 * DEG}"/>
-    <xacro:solid_cylinder
-      name="wheel_${position}_right"
-      length="${wheel_thickness}"
-      radius="${wheel_radius}"
-      roll="${90.0 * DEG}"/>
+      roll="${90.0 * DEG}"
+    />
+    <!-- Juntas contínuas conectando as rodas ao eixo -->
     <xacro:joint_continuous
       name="joint_wheel_${position}_left"
@@ -71,5 +58,7 @@
       child="wheel_${position}_left"
       y="${(wheel_separation + wheel_thickness) * 0.5}"
-      axis="0 1 0"/>
+      axis="0 1 0"
+    />
+    <!-- Juntas contínuas conectando as rodas ao eixo -->
     <xacro:joint_continuous
       name="joint_wheel_${position}_right"
@@ -77,42 +66,51 @@
       child="wheel_${position}_right"
       y="${(wheel_separation + wheel_thickness) * -0.5}"
-      axis="0 1 0"/>
-    <!-- junta fixa para posicionar o axle relativo ao pai (sera usada abaixo) -->
-    <!-- (não cria link adicional aqui — a junta será criada externamente quando necessário) -->
+      axis="0 1 0"
+    />
   </xacro:macro>
-  <!-- Instancia rodas (front e rear). Fornecemos x_offset apenas para documentação; posicionamento feito por joints -->
-  <xacro:wheels position="front" x_offset="${0.5 * wheelbase}"/>
-  <xacro:wheels position="rear"  x_offset="${-0.5 * wheelbase}"/>
-  <!-- Corpo do robô (visual) -->
+  <!-- Instanciação das rodas dianteiras e traseiras -->
+  <xacro:wheels position="front"/>
+  <xacro:wheels position="rear"/>
+  <!-- Definição do corpo do robô -->
   <xacro:solid_block
     name="body"
     size_x="${body_length}"
     size_y="${body_width}"
-    size_z="${body_height}"/>
-  <!-- === Juntas e posicionamento === -->
-  <!-- Posiciona o body em relação ao base_link.
-       Queremos que a origem (0,0,0) do base_link coincida com o eixo traseiro.
-       Então deslocamos o body para frente em +0.5*wheelbase (corpo fica à frente da roda traseira).
-  -->
+    size_z="${body_height}"
+  />
+  <!-- Definição dos para-lamas -->
+  <xacro:solid_block
+    name="fenders_top"
+    size_x="${fender_length}"
+    size_y="${fender_top_width}"
+    size_z="${fender_thickness}"
+    material="Red"
+  />
+  <!-- Juntas fixas conectando os componentes -->
   <xacro:joint_fixed
-    name="joint_base_body"
-    parent="base_link"
-    child="body"
+    parent="body"
+    child="fenders_top"
+    z="${0.5 * (body_height - fender_thickness)}"
+  />
+  <!-- Juntas fixas conectando os eixos das rodas ao corpo -->
+  <xacro:joint_fixed
+    parent="body"
+    child="wheel_front_axle"
     x="${0.5 * wheelbase}"
-    z="${ground_clearance + 0.5 * body_height}"/>
-  <!-- Posiciona o eixo traseiro relativo ao body (visto a partir do body) -->
+    z="${wheel_axle_z_offset}"
+  />
+  <!-- Juntas fixas conectando os eixos das rodas ao corpo -->
   <xacro:joint_fixed
-    name="joint_body_wheel_rear_axle"
     parent="body"
     child="wheel_rear_axle"
     x="${-0.5 * wheelbase}"
-    z="${wheel_axle_z_offset}"/>
-  <!-- Posiciona o eixo dianteiro relativo ao body -->
+    z="${wheel_axle_z_offset}"
+  />
+  <!-- Definição do link base_link como o link raiz -->
+  <link name="base_link"/>
   <xacro:joint_fixed
-    name="joint_body_wheel_front_axle"
-    parent="body"
-    child="wheel_front_axle"
-    x="${0.5 * wheelbase}"
-    z="${wheel_axle_z_offset}"/>
-  <!-- OBS: wheel_*_left/right já estão ligados aos respectivos axle via joint_continuous dentro da macro -->
+    parent="base_link"
+    child="body"
+    z="${ground_clearance + 0.5 * body_height}"
+  />
 </robot>
