Commit message: alteração no arquivo na tentativa de corrigir o robo

File: urdf/rosbot3.xacro (robot description, xacro)
@@ -8,9 +8,10 @@
 <robot name="rosbot3" xmlns:xacro="http://www.ros.org/wiki/xacro">
   <xacro:include filename="$(find rosbot3_description)/urdf/ugv02.xacro"/>
-  <xacro:property name="payload_base_length" value="${156.22 * M}"/>
-  <xacro:property name="payload_base_width" value="${159.96 * M}"/>
-  <xacro:property name="payload_base_height" value="${42.7 * M}"/>
-  <xacro:property name="lidar_side" value="${45.61 * M}"/>
-  <xacro:property name="lidar_height" value="${37.6 * M}"/>
+  <xacro:property name="payload_base_length" value="${10.0 * M}"/>
+  <xacro:property name="payload_base_width" value="${10.0 * M}"/>
+  <xacro:property name="payload_base_height" value="${94.0 * M}"/>
+  <xacro:property name="lidar_size_x" value="${20.0 * M}"/>  <!-- comprimento -->
+  <xacro:property name="lidar_size_y" value="${80.0 * M}"/>   <!-- largura -->
+  <xacro:property name="lidar_size_z" value="${20.0 * M}"/>   <!-- altura -->
   <xacro:solid_block
     name="payload_base"
@@ -20,25 +21,23 @@
   />
   <xacro:joint_fixed
-    parent="body"
+    parent="fenders_top"
     child="payload_base"
-    z="${0.5 * (body_height + payload_base_height)}"
+    x="${-50.0 * M}"
   />
   <xacro:camera_link name="camera_front"/>
   <xacro:joint_fixed
-    parent="payload_base"
+    parent="fenders_top"
     child="camera_front"
-    x="${0.5 * payload_base_length}"
   />
   <xacro:solid_block
     name="lidar"
-    size_x="${lidar_side}"
-    size_y="${lidar_side}"
-    size_z="${lidar_height}"
+    size_x="${lidar_size_x}"
+    size_y="${lidar_size_y}"
+    size_z="${lidar_size_z}"
   />
   <xacro:joint_fixed
     parent="payload_base"
     child="lidar"
-    x="${0.5 * payload_base_height}"
-    z="${0.5 * (payload_base_height + lidar_height)}"
+    z="${payload_base_height * 0.5 + lidar_size_z * 0.5}"
   />
   <link name="laser"/>
@@ -46,5 +45,5 @@
     parent="lidar"
     child="laser"
-    z="${0.5 * lidar_height}"
+    z="${0.5 * lidar_size_z}"
   />
 </robot>

File: urdf/ugv02.xacro (robot description, xacro)
@@ -12,16 +12,15 @@
   <xacro:property name="M" value="0.001"/>
   <xacro:property name="ground_clearance" value="${23.0 * M}"/> <!-- Distância do solo até a parte mais baixa do corpo -->
-  <xacro:property name="overall_height" value="${103 * M}"/> <!-- Altura total do robô -->
-  <xacro:property name="fender_height" value="${10.0 * M}"/> <!-- Altura dos para-lamas -->
-  <xacro:property name="wheel_separation" value="${126.0 * M}"/> <!-- Distância entre as rodas esquerda e direita -->
+  <xacro:property name="overall_height" value="${197 * M}"/> <!-- Altura total do robô -->
+  <xacro:property name="wheel_separation" value="${136.0 * M}"/> <!-- Distância entre as rodas esquerda e direita -->
   <xacro:property name="wheel_diameter" value="${84.0 * M}"/> <!-- Diâmetro das rodas -->
-  <xacro:property name="wheelbase" value="${104.0 * M}"/> <!-- Distância entre os eixos dianteiro e traseiro -->
+  <xacro:property name="wheelbase" value="${116.0 * M}"/> <!-- Distância entre os eixos dianteiro e traseiro -->
   <xacro:property name="wheel_radius" value="${0.5 * wheel_diameter}"/> <!-- Raio das rodas -->
-  <xacro:property name="wheel_thickness" value="${50.21 * M}"/>  <!-- Espessura das rodas -->
+  <xacro:property name="wheel_thickness" value="${50.0 * M}"/>  <!-- Espessura das rodas -->
   <xacro:property name="fender_length" value="${200.0 * M}"/> <!-- Comprimento dos para-lamas -->
-  <xacro:property name="fender_thickness" value="${3.0 * M}"/> <!-- Espessura dos para-lamas -->
+  <xacro:property name="fender_thickness" value="${5.0 * M}"/> <!-- Espessura dos para-lamas -->
   <xacro:property name="fender_top_width" value="${126.0 * M + wheel_thickness}"/> <!-- Largura do para-lama superior -->
   <xacro:property name="body_length" value="${200.0 * M}"/> <!-- Comprimento do corpo do robô -->
-  <xacro:property name="body_width" value="${126.0 * M}"/>
+  <xacro:property name="body_width" value="${126.0 * M}"/> <!-- Largura do corpo do robô -->
   <xacro:property name="body_height" value="${103.0 * M - ground_clearance + 0.004}"/> <!-- Altura do corpo do robô -->
   <xacro:property name="wheel_axle_z_offset" value="${wheel_radius - 0.5 * body_height - ground_clearance}"/>  <!-- Deslocamento Z dos eixos das rodas -->
@@ -31,5 +30,4 @@
     params="position"
   >
-    <!-- Definição das rodas esquerda, direita e do eixo -->
     <xacro:solid_cylinder
       name="wheel_${position}_left"
@@ -38,5 +36,4 @@
       roll="${90.0 * DEG}"
     />
-    <!-- Definição das rodas direita e do eixo -->
     <xacro:solid_cylinder
       name="wheel_${position}_right"
@@ -45,5 +42,4 @@
       roll="${90.0 * DEG}"
     />
-    <!-- Definição do eixo das rodas -->
     <xacro:solid_cylinder
       name="wheel_${position}_axle"
@@ -52,5 +48,4 @@
       roll="${90.0 * DEG}"
     />
-    <!-- Juntas contínuas conectando as rodas ao eixo -->
     <xacro:joint_continuous
       name="joint_wheel_${position}_left"
@@ -60,5 +55,4 @@
       axis="0 1 0"
     />
-    <!-- Juntas contínuas conectando as rodas ao eixo -->
     <xacro:joint_continuous
       name="joint_wheel_${position}_right"
@@ -87,9 +81,22 @@
     material="Red"
   />
+  <!-- Definição do cilindro preto frontal -->
+  <xacro:solid_cylinder
+    name="black_cylinder"
+    radius="${0.5 * wheel_diameter}"
+    length="${38.0 * M}"
+    material="Black"
+  />
+  <!-- Junta fixa conectando o cilindro preto ao para-lama superior -->
+  <xacro:joint_fixed
+    parent="fenders_top"
+    child="black_cylinder"
+    x="${45.0 * M}"
+  />
   <!-- Juntas fixas conectando os componentes -->
   <xacro:joint_fixed
     parent="body"
     child="fenders_top"
-    z="${0.5 * (body_height - fender_thickness)}"
+    z="${body_height*0.5 + fender_thickness*0.5}"
   />
   <!-- Juntas fixas conectando os eixos das rodas ao corpo -->

Commit message: corrigido os erros das rodas do robô e suas dimensões

File: urdf/rosbot3.xacro (robot description, xacro)
@@ -2,15 +2,28 @@
 <!--
   Description of the ROSBOT3 robot.
-  Autor original: Helio Perroni Filho
-  Adaptado por: Vito Rodrigues Franzosi
+  Author: Helio Perroni Filho
+  Adapted by: Vito Rodrigues Franzosi
   Date: 06.11.2025
 -->
 <robot name="rosbot3" xmlns:xacro="http://www.ros.org/wiki/xacro">
   <xacro:include filename="$(find rosbot3_description)/urdf/ugv02.xacro"/>
-  <xacro:property name="payload_base_length" value="${156.22 * M}"/>
-  <xacro:property name="payload_base_width" value="${159.96 * M}"/>
-  <xacro:property name="payload_base_height" value="${42.7 * M}"/>
-  <xacro:property name="lidar_side" value="${45.61 * M}"/>
-  <xacro:property name="lidar_height" value="${37.6 * M}"/>
+  <xacro:property name="payload_base_length" value="${10.0 * M}"/>
+  <xacro:property name="payload_base_width" value="${10.0 * M}"/>
+  <xacro:property name="payload_base_height" value="${120.0 * M}"/>
+  <xacro:property name="lidar_side" value="${20.0 * M}"/>
+  <xacro:property name="lidar_height" value="${80.0 * M}"/>
+  <xacro:property name="cylinder_base_diameter" value="${70.0 * M}"/>
+  <xacro:property name="cylinder_base_height" value="${40.0 * M}"/>
+  <xacro:property name="cylinder_base_radius" value="${cylinder_base_diameter * 0.5}"/>
+  <xacro:solid_cylinder
+    name="cylinder_base"
+    length="${cylinder_base_height}"
+    radius="${cylinder_base_radius}"
+    material="Black"
+  />
+  <xacro:joint_fixed
+    parent="fenders_top"
+    child="cylinder_base"
+  />
   <xacro:solid_block
     name="payload_base"
@@ -18,9 +31,11 @@
     size_y="${payload_base_width}"
     size_z="${payload_base_height}"
+    pitch="${30.0 * DEG}"
   />
   <xacro:joint_fixed
-    parent="body"
+    parent="fenders_top"
     child="payload_base"
-    z="${0.5 * (body_height + payload_base_height)}"
+    x="${(-35.0 * M)}"
+    z="${0.5 * (body_height + fender_thickness)}"
   />
   <xacro:camera_link name="camera_front"/>
@@ -28,17 +43,16 @@
     parent="payload_base"
     child="camera_front"
-    x="${0.5 * payload_base_length}"
   />
   <xacro:solid_block
     name="lidar"
     size_x="${lidar_side}"
-    size_y="${lidar_side}"
-    size_z="${lidar_height}"
+    size_y="${lidar_height}"
+    size_z="${lidar_side}"
   />
   <xacro:joint_fixed
     parent="payload_base"
     child="lidar"
-    x="${0.5 * payload_base_height}"
-    z="${0.5 * (payload_base_height + lidar_height)}"
+    x="${payload_base_width + lidar_side}"
+    z="${0.5 * payload_base_height}"
   />
   <link name="laser"/>

File: urdf/ugv02.xacro (robot description, xacro)
@@ -1,35 +1,36 @@
 <?xml version="1.0" encoding="utf-8"?>
 <!--
-  Modelo simplificado do Waveshare UGV02 (ROSelito) com 4 rodas
-  - Duas dianteiras e duas traseiras
-  - base_link é o link raiz físico (com massa/inércia)
-  Autor original: Helio Perroni Filho
-  Adaptado por: Vito Rodrigues Franzosi
+  Description of the Waveshare UGV02 mobile base upon which ROSBOT3 is built.
+  Author: Helio Perroni Filho
+  Adapted by: Vito Rodrigues Franzosi
   Date: 06.11.2025
 -->
-<robot xmlns:xacro="http://www.ros.org/wiki/xacro"> <!-- Definição do namespace xacro -->
-  <xacro:include filename="$(find ros_commons)/urdf/domain.xacro"/> <!-- Inclui definições de primitivas geométricas -->
+<robot xmlns:xacro="http://www.ros.org/wiki/xacro">
+  <xacro:include filename="$(find ros_commons)/urdf/domain.xacro"/>
   <xacro:property name="M" value="0.001"/>
   <xacro:property name="ground_clearance" value="${23.0 * M}"/> <!-- Distância do solo até a parte mais baixa do corpo -->
-  <xacro:property name="overall_height" value="${103 * M}"/> <!-- Altura total do robô -->
-  <xacro:property name="fender_height" value="${10.0 * M}"/> <!-- Altura dos para-lamas -->
-  <xacro:property name="wheel_separation" value="${126.0 * M}"/> <!-- Distância entre as rodas esquerda e direita -->
-  <xacro:property name="wheel_diameter" value="${84.0 * M}"/> <!-- Diâmetro das rodas -->
-  <xacro:property name="wheelbase" value="${104.0 * M}"/> <!-- Distância entre os eixos dianteiro e traseiro -->
-  <xacro:property name="wheel_radius" value="${0.5 * wheel_diameter}"/> <!-- Raio das rodas -->
-  <xacro:property name="wheel_thickness" value="${50.21 * M}"/>  <!-- Espessura das rodas -->
-  <xacro:property name="fender_length" value="${200.0 * M}"/> <!-- Comprimento dos para-lamas -->
-  <xacro:property name="fender_thickness" value="${3.0 * M}"/> <!-- Espessura dos para-lamas -->
-  <xacro:property name="fender_top_width" value="${126.0 * M + wheel_thickness}"/> <!-- Largura do para-lama superior -->
-  <xacro:property name="body_length" value="${200.0 * M}"/> <!-- Comprimento do corpo do robô -->
-  <xacro:property name="body_width" value="${126.0 * M}"/>
-  <xacro:property name="body_height" value="${103.0 * M - ground_clearance + 0.004}"/> <!-- Altura do corpo do robô -->
-  <xacro:property name="wheel_axle_z_offset" value="${wheel_radius - 0.5 * body_height - ground_clearance}"/>  <!-- Deslocamento Z dos eixos das rodas -->
-  <!-- Definição das rodas -->
+  <xacro:property name="overall_height" value="${141.0 * M}"/> <!-- Altura total do robô -->
+  <xacro:property name="fender_height" value="${10.0 * M}"/>
+  <xacro:property name="wheel_separation" value="${149.0 * M}"/> <!-- Distância entre as rodas esquerda e direita -->
+  <xacro:property name="wheel_diameter" value="${84.0 * M}"/> <!-- Diâmetro da roda -->
+  <xacro:property name="wheelbase" value="${200.0 * M - wheel_diameter}"/> <!-- Distância entre os eixos dianteiro e traseiro -->
+  <xacro:property name="wheel_radius" value="${0.5 * wheel_diameter}"/> <!-- Raio da roda -->
+  <xacro:property name="wheel_thickness" value="${50.0 * M}"/>  <!-- Espessura da roda -->
+  <xacro:property name="fender_length" value="${233.0 * M}"/> <!-- Comprimento dos para-lamas -->
+  <xacro:property name="fender_thickness" value="${3.0 * M}"/>  <!-- Espessura dos para-lamas -->
+  <xacro:property name="fender_top_gap" value="${1.0 * M}"/>  <!-- Espaço entre o topo do para-lama e o corpo -->
+  <xacro:property name="fender_side_gap" value="${5.0 * M}"/> <!-- Espaço entre o lado do para-lama e a roda -->
+  <xacro:property name="body_length" value="${200.0 * M}"/> <!-- Comprimento do corpo -->
+  <xacro:property name="body_width" value="${149.0 * M}"/>  <!-- Largura do corpo -->
+  <xacro:property name="body_height" value="${80.0 * M}"/>
+  <xacro:property name="fender_top_width" value="${body_width + 2.0 * (wheel_thickness + fender_side_gap)}"/>
+  <xacro:property name="fender_side_width" value="${wheel_radius + fender_thickness + fender_top_gap}"/>
+  <xacro:property name="fender_side_y_offset" value="${0.5 * (fender_top_width + fender_thickness)}"/>
+  <xacro:property name="fender_side_z_offset" value="${0.5 * (fender_thickness - fender_side_width)}"/>
+  <xacro:property name="wheel_axle_z_offset" value="${wheel_radius - 0.5 * body_height - ground_clearance}"/>
   <xacro:macro
     name="wheels"
     params="position"
   >
-    <!-- Definição das rodas esquerda, direita e do eixo -->
     <xacro:solid_cylinder
       name="wheel_${position}_left"
@@ -37,6 +38,6 @@
       radius="${wheel_radius}"
       roll="${90.0 * DEG}"
+      material="Black"
     />
-    <!-- Definição das rodas direita e do eixo -->
     <xacro:solid_cylinder
       name="wheel_${position}_right"
@@ -44,6 +45,6 @@
       radius="${wheel_radius}"
       roll="${90.0 * DEG}"
+      material="Black"
     />
-    <!-- Definição do eixo das rodas -->
     <xacro:solid_cylinder
       name="wheel_${position}_axle"
@@ -52,5 +53,4 @@
       roll="${90.0 * DEG}"
     />
-    <!-- Juntas contínuas conectando as rodas ao eixo -->
     <xacro:joint_continuous
       name="joint_wheel_${position}_left"
@@ -60,5 +60,4 @@
       axis="0 1 0"
     />
-    <!-- Juntas contínuas conectando as rodas ao eixo -->
     <xacro:joint_continuous
       name="joint_wheel_${position}_right"
@@ -69,8 +68,6 @@
     />
   </xacro:macro>
-  <!-- Instanciação das rodas dianteiras e traseiras -->
   <xacro:wheels position="front"/>
   <xacro:wheels position="rear"/>
-  <!-- Definição do corpo do robô -->
   <xacro:solid_block
     name="body"
@@ -79,5 +76,4 @@
     size_z="${body_height}"
   />
-  <!-- Definição dos para-lamas -->
   <xacro:solid_block
     name="fenders_top"
@@ -87,11 +83,9 @@
     material="Red"
   />
-  <!-- Juntas fixas conectando os componentes -->
   <xacro:joint_fixed
     parent="body"
     child="fenders_top"
-    z="${0.5 * (body_height - fender_thickness)}"
+    z="${0.5 * (body_height + fender_thickness)}"
   />
-  <!-- Juntas fixas conectando os eixos das rodas ao corpo -->
   <xacro:joint_fixed
     parent="body"
@@ -100,5 +94,4 @@
     z="${wheel_axle_z_offset}"
   />
-  <!-- Juntas fixas conectando os eixos das rodas ao corpo -->
   <xacro:joint_fixed
     parent="body"
@@ -107,5 +100,4 @@
     z="${wheel_axle_z_offset}"
   />
-  <!-- Definição do link base_link como o link raiz -->
   <link name="base_link"/>
   <xacro:joint_fixed

Commit message: alterações nas dimensões do robô

File: urdf/rosbot3.xacro (robot description, xacro)
@@ -60,5 +60,5 @@
     parent="lidar"
     child="laser"
-    z="${0.5 * lidar_size_z}"
+    z="${0.5 * lidar_side}"
   />
 </robot>

File: urdf/ugv02.xacro (robot description, xacro)
@@ -23,10 +23,10 @@
   <xacro:property name="body_length" value="${200.0 * M}"/> <!-- Comprimento do corpo -->
   <xacro:property name="body_width" value="${149.0 * M}"/>  <!-- Largura do corpo -->
-  <xacro:property name="body_height" value="${80.0 * M}"/>
-  <xacro:property name="fender_top_width" value="${body_width + 2.0 * (wheel_thickness + fender_side_gap)}"/>
-  <xacro:property name="fender_side_width" value="${wheel_radius + fender_thickness + fender_top_gap}"/>
-  <xacro:property name="fender_side_y_offset" value="${0.5 * (fender_top_width + fender_thickness)}"/>
-  <xacro:property name="fender_side_z_offset" value="${0.5 * (fender_thickness - fender_side_width)}"/>
-  <xacro:property name="wheel_axle_z_offset" value="${wheel_radius - 0.5 * body_height - ground_clearance}"/>
+  <xacro:property name="body_height" value="${80.0 * M}"/> <!-- Altura do corpo -->
+  <xacro:property name="fender_top_width" value="${body_width + 2.0 * (wheel_thickness + fender_side_gap)}"/> <!-- Largura do topo do para-lama -->
+  <xacro:property name="fender_side_width" value="${wheel_radius + fender_thickness + fender_top_gap}"/> <!-- Largura do lado do para-lama -->
+  <xacro:property name="fender_side_y_offset" value="${0.5 * (fender_top_width + fender_thickness)}"/> <!-- Deslocamento Y do lado do para-lama -->
+  <xacro:property name="fender_side_z_offset" value="${0.5 * (fender_thickness - fender_side_width)}"/> <!-- Deslocamento Z do lado do para-lama -->
+  <xacro:property name="wheel_axle_z_offset" value="${wheel_radius - 0.5 * body_height - ground_clearance}"/> <!-- Deslocamento Z do eixo da roda -->
   <xacro:macro
     name="wheels"
